File: _autosave-MCU.kicad_sch (KiCad schematic)
At the start: 48 parts, among them SW1 RotaryEncoder_Switch, U4 MIC5219-3.3YM5

Commit message: Layout Routing Beign's
Parts:
- removed MT1: PEC11R-4215F-S0024, Rotary_Encoder:RotaryEncoder_Alps_EC11E_Vertical_H20mm, symbol RotaryEncoder:PEC11R-4215F-S0024
- SW1: footprint Rotary_Encoder:RotaryEncoder_Alps_EC11E_Vertical_H20mm -> Rotary_Encoder:RotaryEncoder_Alps_EC12E-Switch_Vertical_H20mm
Changed lines of the file:
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@@
-    )
-  )
-  (symbol (lib_id "RotaryEncoder:PEC11R-4215F-S0024") (at 196.85 73.66 0) (unit 1)
-    (in_bom yes) (on_board yes) (dnp no)
-    (property "Reference" "MT1" (at 196.85 63.5 0)
-      (effects (font (size 1.27 1.27)))
-    )
-    (property "Value" "PEC11R-4215F-S0024" (at 196.85 83.82 0)
-      (effects (font (size 1.27 1.27)))
-    )
-    (property "Footprint" "Rotary_Encoder:RotaryEncoder_Alps_EC11E_Vertical_H20mm" (at 196.85 73.66 0)
-      (effects (font (size 1.27 1.27)) (justify bottom) hide)
-    )
-    (property "Datasheet" "" (at 196.85 73.66 0)
-      (effects (font (size 1.27 1.27)) hide)
-    )
-    (property "MF" "Bourns" (at 196.85 73.66 0)
-      (effects (font (size 1.27 1.27)) (justify bottom) hide)
-    )
-    (property "MAXIMUM_PACKAGE_HEIGHT" "21.5 mm" (at 196.85 73.66 0)
-      (effects (font (size 1.27 1.27)) (justify bottom) hide)
-    )
-    (property "Package" "None" (at 196.85 73.66 0)
-      (effects (font (size 1.27 1.27)) (justify bottom) hide)
-    )
-    (property "Price" "None" (at 196.85 73.66 0)
-      (effects (font (size 1.27 1.27)) (justify bottom) hide)
-    )
-    (property "Check_prices" "https://www.snapeda.com/parts/PEC11R-4215F-S0024/Bourns/view-part/?ref=eda" (at 196.85 73.66 0)
-      (effects (font (size 1.27 1.27)) (justify bottom) hide)
-    )
-    (property "STANDARD" "Manufacturer Recommendations" (at 196.85 73.66 0)
-      (effects (font (size 1.27 1.27)) (justify bottom) hide)
-    )
-    (property "PARTREV" "Rev. 09/19" (at 196.85 73.66 0)
-      (effects (font (size 1.27 1.27)) (justify bottom) hide)
-    )
-    (property "SnapEDA_Link" "https://www.snapeda.com/parts/PEC11R-4215F-S0024/Bourns/view-part/?ref=snap" (at 196.85 73.66 0)
-      (effects (font (size 1.27 1.27)) (justify bottom) hide)
-    )
-    (property "MP" "PEC11R-4215F-S0024" (at 196.85 73.66 0)
-      (effects (font (size 1.27 1.27)) (justify bottom) hide)
-    )
-    (property "Purchase-URL" "https://www.snapeda.com/api/url_track_click_mouser/?unipart_id=428605&manufacturer=Bourns&part_name=PEC11R-4215F-S0024&search_term=None" (at 196.85 73.66 0)
-      (effects (font (size 1.27 1.27)) (justify bottom) hide)
-    )
-    (property "Description" "\nEncoder,Rotary,24 Detents,15 mm, Shaft,Switch | Bourns PEC11R-4215F-S0024\n" (at 196.85 73.66 0)
-      (effects (font (size 1.27 1.27)) (justify bottom) hide)
-    )
-    (property "Availability" "In Stock" (at 196.85 73.66 0)
-      (effects (font (size 1.27 1.27)) (justify bottom) hide)
-    )
-    (property "MANUFACTURER" "J.W.Miller/Bourns" (at 196.85 73.66 0)
-      (effects (font (size 1.27 1.27)) (justify bottom) hide)
-    )
-    (pin "1")
-    (pin "2")
-    (pin "A")
-    (pin "B")
-    (pin "COM")
-    (pin "S1")
-    (pin "S2")
-    (instances
-      (project "Light-CC"
-        (path "/a3254443-8240-44f0-af35-274db02f779b/04c702c6-04db-4682-92c6-1d956531dc1e"
-          (reference "MT1") (unit 1)
-        )
-      )
     )
   )
@@
       (effects (font (size 1.27 1.27)))
     )
-    (property "Footprint" "Rotary_Encoder:RotaryEncoder_Alps_EC11E_Vertical_H20mm" (at 217.17 49.784 0)
+    (property "Footprint" "Rotary_Encoder:RotaryEncoder_Alps_EC12E-Switch_Vertical_H20mm" (at 217.17 49.784 0)
       (effects (font (size 1.27 1.27)) hide)
     )
