File: _autosave-Light-CC.kicad_pcb (KiCad board)
At the start: 2 copper layers, 69 x 36 mm, 69 parts, among them J1 Conn_01x02_Pin, J2 Conn_01x02_Pin, J3 Conn_01x02_Pin, J4 Conn_01x03_Male, J5 USB_C_Receptacle_USB2.0, Q1 BS870, Q2 STD7NK40Z, Q3 BS870, Q4 BC547, Q5 BC547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

Commit message: Layout & routing is almost done Logo need to added
Parts:
- added G***: LOGO, LOGO, F.Cu at (117.2, 104.8)
